Commit message: Current project state, not working teleop

File: urdf/afs_robot.urdf (robot description, URDF)
Before this commit: robot afs_robot, 7 links, 6 joints
Links:
- added link odom
Joints:
- added joint odom_to_base: type fixed, parent odom, child base_link

File: urdf/afs_robot.urdf (copy).xacro (robot description, xacro)
@@ -8,4 +8,7 @@
   <xacro:property name="frame_height" value="0.2" />
   <xacro:property name="articulation_offset" value="0.5" />
+  <!-- В начале файла, где объявляются свойства -->
+	<xacro:property name="wheelbase" value="2.0" />  <!-- Расстояние между осями -->
+	<xacro:property name="articulation_pos" value="${wheelbase*0.1}" />  <!-- Позиция шарнира (0 = середина) -->
   <!-- Предварительные вычисления -->
   <xacro:property name="fl_x" value="${frame_length/2}" />
@@ -25,5 +28,5 @@
 		<parent link="base_link"/>
 		<child link="front_frame"/>
-		<origin xyz="0 0 ${frame_height/2}" rpy="0 0 0"/>
+		<origin xyz="${wheelbase/2} 0 ${frame_height/2}" rpy="0 0 0"/>
 	</joint>
   <!-- Основные рамы -->
@@ -48,12 +51,12 @@
     </visual>
   </link>
-  <!-- Шарнир сочленения -->
-  <joint name="articulation_joint" type="revolute">
-    <parent link="front_frame"/>
-    <child link="rear_frame"/>
-    <origin xyz="${art_x} 0 0" rpy="0 0 0"/>
-    <axis xyz="0 0 1"/>
-    <limit lower="${-pi/4}" upper="${pi/4}" effort="100" velocity="1.0"/>
-  </joint>
+  <!-- Обновлённый шарнир сочленения -->
+	<joint name="articulation_joint" type="revolute">
+		<parent link="front_frame"/>
+		<child link="rear_frame"/>
+		<origin xyz="${-wheelbase/2 + articulation_pos} 0 ${frame_height/2}" rpy="0 0 0"/>
+		<axis xyz="0 0 1"/>
+		<limit lower="-0.8" upper="0.8" effort="100" velocity="1.0"/>
+	</joint>
   <!-- Макрос для колеса с правильной ориентацией -->
   <xacro:macro name="wheel" params="prefix parent x y">

File: urdf/afs_robot.urdf.xacro (robot description, xacro)
@@ -22,4 +22,10 @@
   <xacro:property name="art_x" value="${-(frame_length/2 + articulation_offset)}" />
   <xacro:property name="pi" value="3.1415926535897931" />
+  <!-- Добавим фреймы для одометрии -->
+	<link name="odom"/>
+	<joint name="odom_to_base" type="fixed">
+		<parent link="odom"/>
+		<child link="base_link"/>
+	</joint>
   <!-- Базовый линк (мир) -->
 	<link name="base_link"/>
@@ -118,4 +124,6 @@
       <state_interface name="velocity"/>
     </joint>
+    <state_interface name="front_left_drive_joint/position"/>
+    <state_interface name="front_right_drive_joint/position"/>
   </ros2_control>
 </robot>
